File: mentaldsp.kicad_sch (KiCad schematic)
At the start: 30 parts, among them J1 Conn_PWRJack_2x5.5mm_CUIDevic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, J5 NEMA Conn, J7 NEMA Conn, J8 NEMA Conn, U6 ESP32-S3-SUPERMINI, U7 TMC2209_N0, U8 TMC2209_N2, U9 TMC2209_N1

Commit message: housekeeping
Parts:
- J1: value Conn_PWRJack_2x5.5mm_CUIDevices_PJ-002AH-SMT-TR -> PWRJack
Other:
- company: (none) -> github/thvofi
- title: (none) -> mentaldsp
Changed lines of the file:
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@@
 	(generator_version "10.0")
 	(paper "A4")
+	(title_block
+		(title "mentaldsp")
+		(date "2026-06-01")
+		(rev "v2.0")
+		(company "github/thvofi")
+	)
 	(junction
 		(at 130.81 58.42)
@@
 			)
 		)
-		(property "Value" "Conn_PWRJack_2x5.5mm_CUIDevices_PJ-002AH-SMT-TR"
+		(property "Value" "PWRJack"
 			(at 270.51 147.3199 0)
 			(show_name no)
